File: RemoteEmergencyKill.kicad_pcb (KiCad board)
At the start: 2 copper layers, 35 parts, among them J1 Conn_01x02, J2 Conn_01x02_Female, J3 Conn_01x02_Female, SW1 SW_SPDT, U1 MCP73831-2-OT, U2 ADP151_TSOT, U3 IM920c_ADP_IM920conn

Commit message: complete!!!
Parts:
- removed J3: Conn_01x02_Female, Connector_JST_XA:S02B-XASS-1
- added H1: MountingHole, MountingHole:MountingHole_2.2mm_M2_Pad_Via, F.Cu at (116.8, 71.1)
- BT1: value Battery_Cell -> LP401730; moved to B.Cu
- J2: value Conn_01x02_Female -> Conn_01x03_Female; footprint Connector_JST_XA:S02B-XASS-1 -> Connector_JST_XA:S03B-XASK-1
- moved SW1 72.8 mm to (116.8, 95.2), turned to 270 degrees
- moved J1 62.9 mm to (127.0, 70.5)
- moved JP2 56.8 mm to (127.6, 102.2)
- moved U2 54.4 mm to (125.1, 91.4), turned to 270 degrees
- moved C2 54.3 mm to (124.5, 86.4), turned to 180 degrees
- moved JP12 53.9 mm to (123.3, 102.2), turned to 180 degrees
- moved JP11 49.5 mm to (123.2, 108.6), turned to 270 degrees
- moved JP10 48.3 mm to (140.3, 92.1)
- moved JP1 43.7 mm to (129.5, 108.6), turned to 270 degrees
- moved JP5 41.6 mm to (140.3, 104.8)
- moved R1 41.3 mm to (142.9, 82.5)
- moved R2 40.8 mm to (120.7, 82.5), turned to 90 degrees
- moved D3 40.3 mm to (115.6, 82.5), turned to 90 degrees
- moved R6 40.2 mm to (120.0, 102.2), turned to 270 degrees
- moved D2 39.9 mm to (129.5, 88.3), turned to 90 degrees
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Connections:
- J2 pad 2: GND -> /IO
Routing:
- net /IO: track 0.00 -> 74.2 mm, vias 0 -> 2
- net +5V: track 0.00 -> 47.3 mm, vias 0 -> 2
- net +BATT: track 0.00 -> 38.9 mm, vias 0 -> 1
- net im920_stat: track 0.00 -> 35.6 mm, vias 0 -> 2
- net +3V3: track 0.00 -> 34.3 mm
- net IO8: track 0.00 -> 28.7 mm, vias 0 -> 2
- net chrg_stat: track 0.00 -> 23.4 mm, vias 0 -> 2
- net IO6: track 0.00 -> 22.7 mm, vias 0 -> 2
- net IO7: track 0.00 -> 21.5 mm
- net Reg_in: track 0.00 -> 20.2 mm
- net IO10: track 0.00 -> 17.6 mm, vias 0 -> 2
- net IO4: track 0.00 -> 16.9 mm, vias 0 -> 2
- net Net-(D5-Pad1): track 0.00 -> 15.8 mm, vias 0 -> 2
- net IO5: track 0.00 -> 15.6 mm
- net Net-(D5-Pad2): track 0.00 -> 13.4 mm, vias 0 -> 2
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- added copper zone on B.Cu, net GND
- added copper zone on F.Cu, net GND
Other:
- board outline added: 33 x 52.1 mm
- board text added: "CHRG"
- board text added: "IO state"
- board text added: "IO1 ~~ IO8 IO to Connector"
- board text added: "XCVR"
- board text added: "only Reciever"
- board text added: "only Sender"

Commit message: proted gbr files
Parts:
- moved BT1 15.3 mm to (132.1, 104.1), turned to 180 degrees
Routing:
- net +BATT: track 38.9 -> 13.0 mm
- net /IO: track 74.2 -> 70.2 mm, vias 2 -> 4
- net +5V: track 47.3 -> 50.3 mm, vias 2 -> 0
- net chrg_stat: track 23.4 -> 26.1 mm
Other:
- board text added: "Designed by paripal"
- board text added: "REK-1_0.0"

Commit message: update
Parts:
- U3: value IM920c_ADP_IM920conn -> IM920c; footprint interplan:IM920(IM920c_ADP) -> interplan:IM920c
- moved U3 36.1 mm to (96.0, 110.0), turned to 270 degrees
- moved D5 11.0 mm to (115.6, 97.0)
- moved SW1 5.25 mm to (116.8, 90.0)
- moved D3 5.00 mm to (115.6, 77.5)
- moved D4 5.00 mm to (115.6, 82.6)
- moved R2 5.00 mm to (120.7, 77.5)
- moved R3 5.00 mm to (120.7, 82.6)
Connections:
- U3 pad 15: Net-(U3-Pad15) -> im920_stat
- U3 pad 17: Net-(U3-Pad17) -> +3V3
- U3 pad 18: Net-(U3-Pad18) -> GND
Routing:
- net im920_stat: track 35.6 -> 0.00 mm, vias 2 -> 0
- net IO8: track 28.7 -> 0.00 mm, vias 2 -> 0
- net /IO: track 70.2 -> 43.2 mm, vias 4 -> 2
- net IO6: track 22.7 -> 0.00 mm, vias 2 -> 0
- net IO7: track 21.5 -> 0.00 mm
- net IO10: track 17.6 -> 0.00 mm, vias 2 -> 0
- net IO4: track 16.9 -> 0.00 mm, vias 2 -> 0
- net IO5: track 15.6 -> 0.00 mm
- net EN: track 11.4 -> 0.00 mm
- net +3V3: track 34.3 -> 23.1 mm
- net IO2: track 10.9 -> 0.00 mm, vias 2 -> 0
- net IO3: track 9.98 -> 0.00 mm
- net Reg_in: track 20.2 -> 11.1 mm
- net IO9: track 6.28 -> 0.00 mm
- net Net-(D5-Pad1): track 15.8 -> 11.1 mm
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
Commit message: completed
Parts:
- added J3: Conn_01x02_Female, Connector_JST:JST_XA_S02B-XASK-1_1x02_P2.50mm_Horizontal, F.Cu at (140.3, 78.1)
- J2: value Conn_01x03_Female -> Conn_01x01_Female; footprint Connector_JST_XA:S03B-XASK-1 -> Connector_PinSocket_2.54mm:PinSocket_1x01_P2.54mm_Horizontal
- moved U3 34.2 mm to (130.2, 109.9)
- moved JP10 22.3 mm to (142.2, 114.3), turned to 270 degrees
- moved JP9 19.7 mm to (139.7, 114.3), turned to 270 degrees
- moved JP8 17.4 mm to (137.2, 114.3), turned to 270 degrees
- moved JP3 16.5 mm to (124.5, 114.3), turned to 270 degrees
- moved JP7 15.7 mm to (134.6, 114.3), turned to 270 degrees
- moved JP4 15.1 mm to (127.0, 114.3), turned to 270 degrees
- moved JP6 14.6 mm to (132.1, 114.3), turned to 270 degrees
- moved JP5 14.4 mm to (129.5, 114.3), turned to 270 degrees
- moved R5 8.28 mm to (127.0, 104.1), turned to 0 degrees
- moved JP12 5.46 mm to (127.7, 99.1), turned to 90 degrees
- moved R6 5.46 mm to (124.5, 99.1)
- moved R4 5.12 mm to (131.4, 108.0), turned to 180 degrees
- moved JP2 4.96 mm to (131.4, 99.1), turned to 270 degrees
- moved JP11 4.84 mm to (127.6, 106.7), turned to 0 degrees
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Connections:
- J2 pad 1: +5V -> +3V3
Routing:
- net +3V3: track 23.1 -> 65.1 mm, vias 0 -> 2
- net /IO: track 43.2 -> 84.8 mm, vias 2 -> 1
- net im920_stat: track 0.00 -> 26.9 mm, vias 0 -> 2
- net IO7: track 0.00 -> 26.2 mm, vias 0 -> 2
- net IO8: track 0.00 -> 24.5 mm
- net IO5: track 0.00 -> 20.9 mm, vias 0 -> 2
- net IO6: track 0.00 -> 19.2 mm
- net IO9: track 0.00 -> 16.9 mm, vias 0 -> 2
- net IO3: track 0.00 -> 15.9 mm, vias 0 -> 2
- net IO10: track 0.00 -> 14.3 mm, vias 0 -> 2
- net +5V: track 51.7 -> 37.6 mm
- net IO4: track 0.00 -> 13.9 mm
- net Net-(D5-Pad1): track 11.1 -> 21.9 mm, vias 2 -> 0
- net IO1: track 0.00 -> 9.98 mm
- net IO2: track 0.00 -> 9.31 mm
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