File: RemoteEmergencyKill.sch (KiCad schematic (older format))
At the start: 3 parts

Commit message: schematic update
Parts:
- added BT?: Battery_Cell, symbol Device:Battery_Cell
- added C? (x2): 10u, symbol Device:C
- added D? (x2): D, symbol Device:D
- added R?: R, symbol Device:R
- added U?: MCP1703A-3302_SOT23, Package_TO_SOT_SMD:SOT-23, symbol Regulator_Linear:MCP1703A-3302_SOT23
- added U?: MCP73831-2-OT, Package_TO_SOT_SMD:SOT-23-5, symbol Battery_Management:MCP73831-2-OT
Connections:
- net labels added: +5V, +BATT, Reg_in
- wire segments 8 -> 32
Changed lines of the file:
@@
 EESchema Schematic File Version 4
+LIBS:RemoteEmergencyKill-cache
 EELAYER 30 0
 EELAYER END
@@
 Text Notes 5000 1400 0    50   ~ 0
 mode selecting section
+$Comp
+L Regulator_Linear:MCP1703A-3302_SOT23 U?
+U 1 1 60E1D575
+P 2200 3500
+F 0 "U?" H 2200 3742 50  0000 C CNN
+F 1 "MCP1703A-3302_SOT23" H 2200 3651 50  0000 C CNN
+F 2 "Package_TO_SOT_SMD:SOT-23" H 2200 3700 50  0001 C CNN
+F 3 "http://ww1.microchip.com/downloads/en/DeviceDoc/20005122B.pdf" H 2200 3450 50  0001 C CNN
+	1    2200 3500
+	1    0    0    -1
+$EndComp
+$Comp
+L power:GND #PWR?
+U 1 1 60E20B71
+P 2200 3900
+F 0 "#PWR?" H 2200 3650 50  0001 C CNN
+F 1 "GND" H 2205 3727 50  0000 C CNN
+F 2 "" H 2200 3900 50  0001 C CNN
+F 3 "" H 2200 3900 50  0001 C CNN
+	1    2200 3900
+	1    0    0    -1
+$EndComp
+Wire Wire Line
+	2200 3800 2200 3900
+$Comp
+L Device:C C?
+U 1 1 60E21441
+P 2700 3650
+F 0 "C?" H 2815 3696 50  0000 L CNN
+F 1 "10u" H 2815 3605 50  0000 L CNN
+F 2 "" H 2738 3500 50  0001 C CNN
+F 3 "~" H 2700 3650 50  0001 C CNN
+	1    2700 3650
+	1    0    0    -1
+$EndComp
+$Comp
+L Device:C C?
+U 1 1 60E24981
+P 1700 3650
+F 0 "C?" H 1815 3696 50  0000 L CNN
+F 1 "10u" H 1815 3605 50  0000 L CNN
+F 2 "" H 1738 3500 50  0001 C CNN
+F 3 "~" H 1700 3650 50  0001 C CNN
+	1    1700 3650
+	1    0    0    -1
+$EndComp
+Wire Wire Line
+	1900 3500 1700 3500
+Wire Wire Line
+	1700 3800 1700 3900
+Wire Wire Line
+	1700 3900 2200 3900
+Connection ~ 2200 3900
+Wire Wire Line
+	2500 3500 2700 3500
+Wire Wire Line
+	2700 3800 2700 3900
+Wire Wire Line
+	2700 3900 2200 3900
+$Comp
+L Device:D D?
+U 1 1 60E25521
+P 1350 3500
+F 0 "D?" H 1350 3283 50  0000 C CNN
+F 1 "D" H 1350 3374 50  0000 C CNN
+F 2 "" H 1350 3500 50  0001 C CNN
+F 3 "~" H 1350 3500 50  0001 C CNN
+	1    1350 3500
+	-1   0    0    1
+$EndComp
+Wire Wire Line
+	1700 3500 1500 3500
+Connection ~ 1700 3500
+Wire Wire Line
+	2700 3500 2800 3500
+Wire Wire Line
+	2800 3500 2800 3400
+Connection ~ 2700 3500
+$Comp
+L power:+3.3V #PWR?
+U 1 1 60E2741F
+P 2800 3400
+F 0 "#PWR?" H 2800 3250 50  0001 C CNN
+F 1 "+3.3V" H 2815 3573 50  0000 C CNN
+F 2 "" H 2800 3400 50  0001 C CNN
+F 3 "" H 2800 3400 50  0001 C CNN
+	1    2800 3400
+	1    0    0    -1
+$EndComp
+$Comp
+L Battery_Management:MCP73831-2-OT U?
+U 1 1 60E27F6E
+P 1750 1700
+F 0 "U?" H 1750 2181 50  0000 C CNN
+F 1 "MCP73831-2-OT" H 1750 2090 50  0000 C CNN
+F 2 "Package_TO_SOT_SMD:SOT-23-5" H 1800 1450 50  0001 L CIN
+F 3 "http://ww1.microchip.com/downloads/en/DeviceDoc/20001984g.pdf" H 1600 1650 50  0001 C CNN
+	1    1750 1700
+	1    0    0    -1
+$EndComp
+$Comp
+L Device:Battery_Cell BT?
+U 1 1 60E33702
+P 2550 1800
+F 0 "BT?" H 2668 1896 50  0000 L CNN
+F 1 "Battery_Cell" H 2668 1805 50  0000 L CNN
+F 2 "" V 2550 1860 50  0001 C CNN
+F 3 "~" V 2550 1860 50  0001 C CNN
+	1    2550 1800
+	1    0    0    -1
+$EndComp
+Wire Wire Line
+	2150 1600 2550 1600
+Wire Wire Line
+	2550 1900 2550 2100
+Wire Wire Line
+	2550 2100 1750 2100
+Wire Wire Line
+	1750 2100 1750 2000
+Wire Wire Line
+	1750 2100 1750 2200
+Connection ~ 1750 2100
+$Comp
+L power:GND #PWR?
+U 1 1 60E365AF
+P 1750 2200
+F 0 "#PWR?" H 1750 1950 50  0001 C CNN
+F 1 "GND" H 1755 2027 50  0000 C CNN
+F 2 "" H 1750 2200 50  0001 C CNN
+F 3 "" H 1750 2200 50  0001 C CNN
+	1    1750 2200
+	1    0    0    -1
+$EndComp
+Wire Wire Line
+	2550 1600 2650 1600
+Connection ~ 2550 1600
+Wire Wire Line
+	2650 1600 2650 1500
+$Comp
+L power:+BATT #PWR?
+U 1 1 60E37A51
+P 2650 1500
+F 0 "#PWR?" H 2650 1350 50  0001 C CNN
+F 1 "+BATT" H 2665 1673 50  0000 C CNN
+F 2 "" H 2650 1500 50  0001 C CNN
+F 3 "" H 2650 1500 50  0001 C CNN
+	1    2650 1500
+	1    0    0    -1
+$EndComp
+$Comp
+L Device:D D?
+U 1 1 60E38EF6
+P 1700 3250
+F 0 "D?" H 1700 3033 50  0000 C CNN
+F 1 "D" H 1700 3124 50  0000 C CNN
+F 2 "" H 1700 3250 50  0001 C CNN
+F 3 "~" H 1700 3250 50  0001 C CNN
+	1    1700 3250
+	0    -1   -1   0
+$EndComp
+Wire Wire Line
+	1700 3400 1700 3500
+$Comp
+L power:+5V #PWR?
+U 1 1 60E39C29
+P 1700 3000
+F 0 "#PWR?" H 1700 2850 50  0001 C CNN
+F 1 "+5V" H 1715 3173 50  0000 C CNN
+F 2 "" H 1700 3000 50  0001 C CNN
+F 3 "" H 1700 3000 50  0001 C CNN
+	1    1700 3000
+	1    0    0    -1
+$EndComp
+Wire Wire Line
+	1700 3000 1700 3100
+$Comp
+L power:+5V #PWR?
+U 1 1 60E3B875
+P 1750 1300
+F 0 "#PWR?" H 1750 1150 50  0001 C CNN
+F 1 "+5V" H 1765 1473 50  0000 C CNN
+F 2 "" H 1750 1300 50  0001 C CNN
+F 3 "" H 1750 1300 50  0001 C CNN
+	1    1750 1300
+	1    0    0    -1
+$EndComp
+Wire Wire Line
+	1750 1300 1750 1400
+$Comp
+L Device:R R?
+U 1 1 60E3C1F9
+P 1150 1950
+F 0 "R?" H 1220 1996 50  0000 L CNN
+F 1 "R" H 1220 1905 50  0000 L CNN
+F 2 "" V 1080 1950 50  0001 C CNN
+F 3 "~" H 1150 1950 50  0001 C CNN
+	1    1150 1950
+	1    0    0    -1
+$EndComp
+Wire Wire Line
+	1350 1800 1150 1800
+Wire Wire Line
+	1150 2100 1750 2100
+Wire Wire Line
+	1200 3500 1100 3500
+$Comp
+L power:+BATT #PWR?
+U 1 1 60E3EA5A
+P 1100 3000
+F 0 "#PWR?" H 1100 2850 50  0001 C CNN
+F 1 "+BATT" H 1115 3173 50  0000 C CNN
+F 2 "" H 1100 3000 50  0001 C CNN
+F 3 "" H 1100 3000 50  0001 C CNN
+	1    1100 3000
+	1    0    0    -1
+$EndComp
+Wire Wire Line
+	1100 3000 1100 3500
+Text Label 1700 3500 0    50   ~ 0
+Reg_in
 $EndSCHEMATC

Commit message: changed regulator
Parts:
- removed U?: MCP1703A-3302_SOT23, Package_TO_SOT_SMD:SOT-23, symbol Regulator_Linear:MCP1703A-3302_SOT23
- added C? (x2): 10u, Capacitor_SMD:C_0805_2012Metric, symbol Device:C
- added D? (x3): LED, LED_SMD:LED_0603_1608Metric, symbol Device:LED
- added J?: Conn_01x02, Connector_USB_additional:USB micro B 2pin, symbol Connector_Generic:Conn_01x02
- added J? (x2): Conn_01x02_Female, Connector_JST_XA:S02B-XASS-1, symbol Connector:Conn_01x02_Female
- added JP? (x10): SolderJumper_2_Open, Jumper:SolderJumper-2_P1.3mm_Open_TrianglePad1.0x1.5mm, symbol Jumper:SolderJumper_2_Open
- added R?: 10k, Resistor_SMD:R_0603_1608Metric, symbol Device:R
- added R? (x2): 330, Resistor_SMD:R_0603_1608Metric, symbol Device:R
- added R? (x2): 1k, Resistor_SMD:R_0603_1608Metric, symbol Device:R
- added U?: ADP151_TSOT, Package_TO_SOT_SMD:TSOT-23-5, symbol AnalogDevices:ADP151_TSOT
- C? (x2): footprint (none) -> Capacitor_SMD:C_0805_2012Metric
- D? (x2): footprint (none) -> Diode_SMD:D_SOD-123F
- JP? (x2): footprint (none) -> Jumper:SolderJumper-2_P1.3mm_Open_TrianglePad1.0x1.5mm
- R?: value R -> R_chrg_prog; footprint (none) -> Resistor_SMD:R_0603_1608Metric
Connections:
- net labels added: EN, IO, IO1, IO2, IO3, IO4, IO5, IO6, IO7, IO8, chrg_stat, im920_stat
- net labels removed: STATUS
- wire segments 32 -> 93
Other:
- note added: "USB_2pin_pw"
- note added: "XA_2pin_SW_or_OUT"
- note added: "XA_2pin_pw"
- note added: "mode selecting"
- note added: "only_OUT"
- note added: "only_SW"
- note removed: "mode selecting section"
- moved on the sheet: BT?, C?

Commit message: pcb file added
Parts:
- added SW1: SW_SPDT, Button_Switch_additional:IS-1245T-G, symbol Switch:SW_SPDT
- BT1: renamed from BT?; footprint (none) -> Battery_additional:LP401730
- R1: renamed from R?; value R_chrg_prog -> 10k
- gave numbers to parts that had none: 32
Connections:
- net EN: now also SW1.2 (B)
- net GND: now also SW1.3 (C)
- net Reg_in: now also SW1.1 (A)
- net RESET: no longer names the net of U3.25 (RESET)
Other:
- moved on the sheet: D1

Commit message: complete!!!
Parts:
- removed J2, J3: Conn_01x02_Female, Connector_JST_XA:S02B-XASS-1, symbol Connector:Conn_01x02_Female
- added H1: MountingHole, MountingHole:MountingHole_2.2mm_M2_Pad_Via, symbol Mechanical:MountingHole
- added J2: Conn_01x03_Female, Connector_JST_XA:S03B-XASK-1, symbol Connector:Conn_01x03_Female
- BT1: value Battery_Cell -> LP401730
Connections:
- net +5V: now also J2.1 (Pin_1)
- net GND: now also J2.3 (Pin_3)
- net IO: now also J2.2 (Pin_2)
Changed lines of the file:
@@
 im920_stat
 $Comp
-L power:GND #PWR012
+L power:GND #PWR013
 U 1 1 60E1495C
 P 6200 4200
-F 0 "#PWR012" H 6200 3950 50  0001 C CNN
+F 0 "#PWR013" H 6200 3950 50  0001 C CNN
 F 1 "GND" H 6205 4027 50  0000 C CNN
 F 2 "" H 6200 4200 50  0001 C CNN
@@
 	4450 4000 4450 3800
 $Comp
-L power:+3.3V #PWR010
+L power:+3.3V #PWR011
 U 1 1 60E16909
 P 4450 3800
-F 0 "#PWR010" H 4450 3650 50  0001 C CNN
+F 0 "#PWR011" H 4450 3650 50  0001 C CNN
 F 1 "+3.3V" H 4465 3973 50  0000 C CNN
 F 2 "" H 4450 3800 50  0001 C CNN
@@
 $EndComp
 $Comp
-L power:+3.3V #PWR011
+L power:+3.3V #PWR012
 U 1 1 60E181F9
 P 5050 1700
-F 0 "#PWR011" H 5050 1550 50  0001 C CNN
+F 0 "#PWR012" H 5050 1550 50  0001 C CNN
 F 1 "+3.3V" H 5065 1873 50  0000 C CNN
 F 2 "" H 5050 1700 50  0001 C CNN
@@
 P 3000 1800
 F 0 "BT1" H 3118 1896 50  0000 L CNN
-F 1 "Battery_Cell" H 3118 1805 50  0000 L CNN
+F 1 "LP401730" H 3118 1805 50  0000 L CNN
 F 2 "Battery_additional:LP401730" V 3000 1860 50  0001 C CNN
 F 3 "~" V 3000 1860 50  0001 C CNN
@@
 $EndComp
 $Comp
-L power:+5V #PWR014
+L power:+5V #PWR015
 U 1 1 60E4165C
 P 8150 1350
-F 0 "#PWR014" H 8150 1200 50  0001 C CNN
+F 0 "#PWR015" H 8150 1200 50  0001 C CNN
 F 1 "+5V" H 8165 1523 50  0000 C CNN
 F 2 "" H 8150 1350 50  0001 C CNN
@@
 	8150 1550 8150 1650
 $Comp
-L power:GND #PWR015
+L power:GND #PWR016
 U 1 1 60E43088
 P 8150 1650
-F 0 "#PWR015" H 8150 1400 50  0001 C CNN
+F 0 "#PWR016" H 8150 1400 50  0001 C CNN
 F 1 "GND" H 8155 1477 50  0000 C CNN
 F 2 "" H 8150 1650 50  0001 C CNN
@@
 $EndComp
 $Comp
-L Connector:Conn_01x02_Female J2
-U 1 1 60E437D8
-P 8500 2450
-F 0 "J2" H 8528 2426 50  0000 L CNN
-F 1 "Conn_01x02_Female" H 8528 2335 50  0000 L CNN
-F 2 "Connector_JST_XA:S02B-XASS-1" H 8500 2450 50  0001 C CNN
-F 3 "~" H 8500 2450 50  0001 C CNN
-	1    8500 2450
-	1    0    0    -1
-$EndComp
-$Comp
-L power:+5V #PWR016
+L power:+5V #PWR017
 U 1 1 60E45A91
-P 8150 2350
-F 0 "#PWR016" H 8150 2200 50  0001 C CNN
-F 1 "+5V" H 8165 2523 50  0000 C CNN
-F 2 "" H 8150 2350 50  0001 C CNN
-F 3 "" H 8150 2350 50  0001 C CNN
-	1    8150 2350
-	1    0    0    -1
-$EndComp
-Wire Wire Line
-	8300 2450 8150 2450
-Wire Wire Line
-	8150 2450 8150 2350
-Wire Wire Line
-	8300 2550 8150 2550
-Wire Wire Line
-	8150 2550 8150 2650
-$Comp
-L power:GND #PWR017
-U 1 1 60E45A9B
-P 8150 2650
-F 0 "#PWR017" H 8150 2400 50  0001 C CNN
-F 1 "GND" H 8155 2477 50  0000 C CNN
-F 2 "" H 8150 2650 50  0001 C CNN
-F 3 "" H 8150 2650 50  0001 C CNN
-	1    8150 2650
-	1    0    0    -1
-$EndComp
+P 8650 4250
+F 0 "#PWR017" H 8650 4100 50  0001 C CNN
+F 1 "+5V" H 8665 4423 50  0000 C CNN
+F 2 "" H 8650 4250 50  0001 C CNN
+F 3 "" H 8650 4250 50  0001 C CNN
+	1    8650 4250
+	1    0    0    -1
+$EndComp
+Wire Wire Line
+	8800 4350 8650 4350
+Wire Wire Line
+	8650 4350 8650 4250
 Text Notes 8500 1350 0    50   ~ 0
 USB_2pin_pw
@@
 Connection ~ 8000 3450
 $Comp
-L power:+3.3V #PWR013
+L power:+3.3V #PWR014
 U 1 1 60E8B713
 P 8000 3350
-F 0 "#PWR013" H 8000 3200 50  0001 C CNN
+F 0 "#PWR014" H 8000 3200 50  0001 C CNN
 F 1 "+3.3V" H 8015 3523 50  0000 C CNN
 F 2 "" H 8000 3350 50  0001 C CNN
@@
 	3500 2200 3500 2300
 $Comp
-L power:+5V #PWR08
+L power:+5V #PWR09
 U 1 1 60E99C0D
 P 3500 1500
-F 0 "#PWR08" H 3500 1350 50  0001 C CNN
+F 0 "#PWR09" H 3500 1350 50  0001 C CNN
 F 1 "+5V" H 3515 1673 50  0000 C CNN
 F 2 "" H 3500 1500 50  0001 C CNN
@@
 Text Notes 9000 4350 0    50   ~ 0
 XA_2pin_SW_or_OUT
-$Comp
-L Connector:Conn_01x02_Female J3
-U 1 1 60E4894D
-P 9000 4450
-F 0 "J3" H 9028 4426 50  0000 L CNN
-F 1 "Conn_01x02_Female" H 9028 4335 50  0000 L CNN
-F 2 "Connector_JST_XA:S02B-XASS-1" H 9000 4450 50  0001 C CNN
-F 3 "~" H 9000 4450 50  0001 C CNN
-	1    9000 4450
-	1    0    0    -1
-$EndComp
 Wire Wire Line
 	8000 4450 8800 4450
@@
 Connection ~ 1150 2100
 $Comp
-L power:GND #PWR09
+L power:GND #PWR010
 U 1 1 60EFC176
 P 4000 2300
-F 0 "#PWR09" H 4000 2050 50  0001 C CNN
+F 0 "#PWR010" H 4000 2050 50  0001 C CNN
 F 1 "GND" H 4005 2127 50  0000 C CNN
 F 2 "" H 4000 2300 50  0001 C CNN
@@
 Reg_in
 $Comp
-L power:GND #PWR020
+L power:GND #PWR08
 U 1 1 60E7602C
 P 3300 4700
-F 0 "#PWR020" H 3300 4450 50  0001 C CNN
+F 0 "#PWR08" H 3300 4450 50  0001 C CNN
 F 1 "GND" H 3305 4527 50  0000 C CNN
 F 2 "" H 3300 4700 50  0001 C CNN
@@
 Wire Wire Line
 	3300 4600 3300 4700
+$Comp
+L Connector:Conn_01x03_Female J2
+U 1 1 60E792F1
+P 9000 4450
+F 0 "J2" H 9028 4476 50  0000 L CNN
+F 1 "Conn_01x03_Female" H 9028 4385 50  0000 L CNN
+F 2 "Connector_JST_XA:S03B-XASK-1" H 9000 4450 50  0001 C CNN
+F 3 "~" H 9000 4450 50  0001 C CNN
+	1    9000 4450
+	1    0    0    -1
+$EndComp
+$Comp
+L Mechanical:MountingHole H1
+U 1 1 60EB1A83
+P 9500 1000
+F 0 "H1" H 9600 1046 50  0000 L CNN
+F 1 "MountingHole" H 9600 955 50  0000 L CNN
+F 2 "MountingHole:MountingHole_2.2mm_M2_Pad_Via" H 9500 1000 50  0001 C CNN
+F 3 "~" H 9500 1000 50  0001 C CNN
+	1    9500 1000
+	1    0    0    -1
+$EndComp
 $EndSCHEMATC

Commit message: chenge schematic
Parts:
- removed U3: IM920c_ADP_IM920conn, interplan:IM920(IM920c_ADP), symbol interplan:IM920c_ADP_IM920conn
- added U?: IM920c, interplan:IM920c, symbol interplan:IM920c
Connections:
- net +3V3: now also U?.17 (VCC)
- net GND: now also U?.18 (GND)
- net IO1: now also U?.1 (IO1/RTS)
- net IO10: now also U?.10 (IO10)
- net IO2: now also U?.2 (IO2)
- net IO3: now also U?.3 (IO3)
- net IO4: now also U?.4 (IO4)
- net IO5: now also U?.5 (IO5)
- net IO6: now also U?.6 (IO6/RxD)
- net IO7: now also U?.7 (IO7/TxD)
- net IO8: now also U?.8 (IO8)
- net IO9: now also U?.9 (IO9)
- net im920_stat: now also U?.15 (STATUS)
Changed lines of the file:
@@
 Comment4 ""
 $EndDescr
-$Comp
-L interplan:IM920c_ADP_IM920conn U3
-U 1 1 60E09FCC
-P 5500 3250
-F 0 "U3" H 5500 3915 50  0000 C CNN
-F 1 "IM920c_ADP_IM920conn" H 5500 3824 50  0000 C CNN
-F 2 "interplan:IM920(IM920c_ADP)" H 5500 3800 50  0001 C CNN
-F 3 "https://www.interplan.co.jp/support/solution/IM315/manual/IM920c_ADP_manual.pdf" H 5500 3800 50  0001 C CNN
-	1    5500 3250
-	1    0    0    -1
-$EndComp
 Text GLabel 5000 3300 0    50   Input ~ 0
 IO9
 Text GLabel 6000 3300 2    50   Input ~ 0
 IO10
-Text GLabel 5000 3900 0    50   Input ~ 0
+Text GLabel 5000 3600 0    50   Input ~ 0
 im920_stat
 $Comp
 L power:GND #PWR013
 U 1 1 60E1495C
-P 6200 4200
-F 0 "#PWR013" H 6200 3950 50  0001 C CNN
-F 1 "GND" H 6205 4027 50  0000 C CNN
-F 2 "" H 6200 4200 50  0001 C CNN
-F 3 "" H 6200 4200 50  0001 C CNN
-	1    6200 4200
-	1    0    0    -1
-$EndComp
-Wire Wire Line
-	6200 4200 6200 4000
-Wire Wire Line
-	6200 4000 6000 4000
-Wire Wire Line
-	5000 4000 4450 4000
-Wire Wire Line
-	4450 4000 4450 3800
+P 6200 3900
+F 0 "#PWR013" H 6200 3650 50  0001 C CNN
+F 1 "GND" H 6205 3727 50  0000 C CNN
+F 2 "" H 6200 3900 50  0001 C CNN
+F 3 "" H 6200 3900 50  0001 C CNN
+	1    6200 3900
+	1    0    0    -1
+$EndComp
+Wire Wire Line
+	6200 3900 6200 3700
+Wire Wire Line
+	6200 3700 6000 3700
+Wire Wire Line
+	5000 3700 4450 3700
+Wire Wire Line
+	4450 3700 4450 3500
 $Comp
 L power:+3.3V #PWR011
 U 1 1 60E16909
-P 4450 3800
-F 0 "#PWR011" H 4450 3650 50  0001 C CNN
-F 1 "+3.3V" H 4465 3973 50  0000 C CNN
-F 2 "" H 4450 3800 50  0001 C CNN
-F 3 "" H 4450 3800 50  0001 C CNN
-	1    4450 3800
+P 4450 3500
+F 0 "#PWR011" H 4450 3350 50  0001 C CNN
+F 1 "+3.3V" H 4465 3673 50  0000 C CNN
+F 2 "" H 4450 3500 50  0001 C CNN
+F 3 "" H 4450 3500 50  0001 C CNN
+	1    4450 3500
 	1    0    0    -1
 $EndComp
@@
 	1    0    0    -1
 $EndComp
+$Comp
+L interplan:IM920c U?
+U 1 1 612751ED
+P 5500 3250
+F 0 "U?" H 5500 3915 50  0000 C CNN
+F 1 "IM920c" H 5500 3824 50  0000 C CNN
+F 2 "interplan:IM920c" H 5500 3800 50  0001 C CNN
+F 3 "" H 5500 3800 50  0001 C CNN
+	1    5500 3250
+	1    0    0    -1
+$EndComp

Commit message: update
Parts:
- gave numbers to parts that had none: 1
Changed lines of the file:
@@
 $EndComp
 $Comp
-L interplan:IM920c U?
+L interplan:IM920c U3
 U 1 1 612751ED
 P 5500 3250
-F 0 "U?" H 5500 3915 50  0000 C CNN
+F 0 "U3" H 5500 3915 50  0000 C CNN
 F 1 "IM920c" H 5500 3824 50  0000 C CNN
 F 2 "interplan:IM920c" H 5500 3800 50  0001 C CNN

Commit message: completed
Parts:
- removed J2: Conn_01x03_Female, Connector_JST_XA:S03B-XASK-1, symbol Connector:Conn_01x03_Female
- added J2: Conn_01x01_Female, Connector_PinSocket_2.54mm:PinSocket_1x01_P2.54mm_Horizontal, symbol Connector:Conn_01x01_Female
- added J3: Conn_01x02_Female, Connector_JST:JST_XA_S02B-XASK-1_1x02_P2.50mm_Horizontal, symbol Connector:Conn_01x02_Female
Connections:
- net +3V3: now also J2.1 (Pin_1)
- net GND: now also J3.2 (Pin_2)
- net IO: now also J3.1 (Pin_1)
Changed lines of the file:
@@
 EESchema Schematic File Version 4
-LIBS:RemoteEmergencyKill-cache
 EELAYER 30 0
 EELAYER END
@@
 	1    0    0    -1
 $EndComp
-$Comp
-L power:+5V #PWR017
-U 1 1 60E45A91
-P 8650 4250
-F 0 "#PWR017" H 8650 4100 50  0001 C CNN
-F 1 "+5V" H 8665 4423 50  0000 C CNN
-F 2 "" H 8650 4250 50  0001 C CNN
-F 3 "" H 8650 4250 50  0001 C CNN
-	1    8650 4250
-	1    0    0    -1
-$EndComp
 Wire Wire Line
 	8800 4350 8650 4350
@@
 	3300 4600 3300 4700
 $Comp
-L Connector:Conn_01x03_Female J2
-U 1 1 60E792F1
-P 9000 4450
-F 0 "J2" H 9028 4476 50  0000 L CNN
-F 1 "Conn_01x03_Female" H 9028 4385 50  0000 L CNN
-F 2 "Connector_JST_XA:S03B-XASK-1" H 9000 4450 50  0001 C CNN
-F 3 "~" H 9000 4450 50  0001 C CNN
-	1    9000 4450
-	1    0    0    -1
-$EndComp
-$Comp
 L Mechanical:MountingHole H1
 U 1 1 60EB1A83
@@
 	1    0    0    -1
 $EndComp
+$Comp
+L power:+3.3V #PWR017
+U 1 1 61275944
+P 8650 4250
+F 0 "#PWR017" H 8650 4100 50  0001 C CNN
+F 1 "+3.3V" H 8665 4423 50  0000 C CNN
+F 2 "" H 8650 4250 50  0001 C CNN
+F 3 "" H 8650 4250 50  0001 C CNN
+	1    8650 4250
+	1    0    0    -1
+$EndComp
+$Comp
+L Connector:Conn_01x02_Female J3
+U 1 1 612783C8
+P 9000 4450
+F 0 "J3" H 9028 4426 50  0000 L CNN
+F 1 "Conn_01x02_Female" H 9028 4335 50  0000 L CNN
+F 2 "Connector_JST:JST_XA_S02B-XASK-1_1x02_P2.50mm_Horizontal" H 9000 4450 50  0001 C CNN
+F 3 "~" H 9000 4450 50  0001 C CNN
+	1    9000 4450
+	1    0    0    -1
+$EndComp
+$Comp
+L Connector:Conn_01x01_Female J2
+U 1 1 612791FB
+P 9000 4350
+F 0 "J2" H 9028 4376 50  0000 L CNN
+F 1 "Conn_01x01_Female" H 9028 4285 50  0000 L CNN
+F 2 "Connector_PinSocket_2.54mm:PinSocket_1x01_P2.54mm_Horizontal" H 9000 4350 50  0001 C CNN
+F 3 "~" H 9000 4350 50  0001 C CNN
+	1    9000 4350
+	1    0    0    -1
+$EndComp
